Commit message: wheels added

File: urdf/right_left_wheel.urdf (robot description, URDF)
Before this commit: robot guru_bot, 3 links, 2 joints
Links:
- added link left_wheel; visual cylinder length=0.075 radius=0.055
- added link right_wheel; visual cylinder length=0.075 radius=0.055
Joints:
- added joint left_wheel_joint: type continuous, parent base_link, child left_wheel, origin xyz=-0.2825 .13 -.05 rpy=-1.5707 0.0 0.0, axis 0.0 0.0 1.0
- added joint right_wheel_joint: type continuous, parent base_link, child right_wheel, origin xyz=-0.2825 -.13 -.05 rpy=-1.5707 0.0 0.0, axis 0.0 0.0 1.0

Commit message: Physical Props added (Collision, Inertia)

File: urdf/right_left_wheel.urdf (robot description, URDF)
Before this commit: robot guru_bot, 5 links, 4 joints
Links:
- link base_link: mass None -> 2; geometry collision box size=0.6 0.3 0.1; visual box size=0.6 0.3 0.1
- link front_caster_of_wheel: mass None -> 0.1; geometry collision box size=0.1 0.1 0.1; visual box size=0.1 0.1 0.1
- link front_wheel: mass None -> 0.1; geometry collision cylinder length=0.05 radius=0.035; visual cylinder length=0.05 radius=0.035
- link left_wheel: mass None -> 0.1; geometry collision cylinder length=0.075 radius=0.055; visual cylinder length=0.075 radius=0.055
- link right_wheel: mass None -> 0.1; geometry collision cylinder length=0.075 radius=0.055; visual cylinder length=0.075 radius=0.055

Commit message: Innertia corrected

File: urdf/right_left_wheel.urdf (robot description, URDF)
Before this commit: robot guru_bot, 5 links, 4 joints
Links:
- link base_link: mass 2 -> 1.0
